File: EDA_designs/microfluidics-chip.kicad_pcb (KiCad board)
At the start: 4 copper layers, 78 x 78 mm, 39 parts, among them J1 Conn_01x06_Pin, J10 39-53-2045, J11 Conn_01x14_Pin, J12 Conn_01x14_Pin, J13 39-53-2045, J14 39-53-2045, J15 Conn_ARM_SWD_TagConnect_TC2030, J16 Conn_01x02_Socket, J18 EJ508A, J2 Conn_01x06_Pin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

Commit message: Pushing v3
Parts:
- J1, J2, J3, J4: value Conn_01x06_Pin -> 532610671; footprint Connector_Hirose:Hirose_DF13-06P-1.25DSA_1x06_P1.25mm_Vertical -> co2_sensor_footprint:CON_532610671
- moved J1 26.2 mm to (187.1, 115.5), turned to 90 degrees
- moved J4 19.0 mm to (196.2, 94.9), turned to 90 degrees
- moved J3 15.0 mm to (196.1, 115.5), turned to 90 degrees
- moved J2 6.89 mm to (187.1, 94.8), turned to 90 degrees
- moved G*** 1.92 mm to (179.5, 74.0)
Connections:
- J3 pad 1: /IRQn1 -> /IRQn2
- J4 pad 1: /IRQn2 -> /IRQn1
Routing:
- net /IRQn3: track 147.1 -> 118.7 mm
- net /I2C_SDA: track 123.1 -> 137.5 mm, vias 0 -> 6
- net /IRQn1: track 145.6 -> 159.1 mm
- net /IRQn4: track 132.7 -> 138.4 mm, vias 0 -> 2
- net /I2C_SCK: track 132.9 -> 128.8 mm
- net /IRQn2: track 131.3 -> 128.9 mm
- net GND: vias 17 -> 29
- net +3.3V: vias 10 -> 14
Other:
- board size 78 x 78 mm -> 86.5 x 78 mm
- board text added: "8/11/24 | Rev. 3"
- board text removed: "8/10/24 | Rev. 2"

Commit message: v4
Parts:
- moved J2 24.4 mm to (199.1, 116.1), turned to 180 degrees
- moved J3 17.6 mm to (199.0, 98.1), turned to 180 degrees
- moved J1 14.6 mm to (199.1, 107.1), turned to 180 degrees
- moved J4 6.59 mm to (199.1, 88.9), turned to 180 degrees
Routing:
- net /IRQn2: track 128.9 -> 159.6 mm
- net /IRQn3: track 118.7 -> 148.6 mm
- net /I2C_SDA: track 137.5 -> 164.1 mm, vias 6 -> 5
- net /IRQn1: track 159.1 -> 171.3 mm
- net /IRQn4: track 138.4 -> 126.8 mm, vias 2 -> 0
- net /I2C_SCK: track 128.8 -> 135.4 mm
- net GND: vias 29 -> 27
Other:
- board size 86.5 x 78 mm -> 90 x 78 mm
- board text added: "8/11/24 | Rev. 4"
- board text removed: "8/11/24 | Rev. 3"
