File: EDA_designs/ion-concentration-biomodulator.kicad_sch (KiCad schematic)
At the start: 39 parts, among them J1 532610671, J10 39-53-2045, J11 Conn_01x14_Pin, J12 Conn_01x14_Pin, J13 39-53-2045, J14 39-53-2045, J15 Conn_ARM_SWD_TagConnect_TC2030, J16 Conn_01x02_Socket, J18 EJ508A, J2 532610671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

Commit message: pushing v5
Parts:
- removed C11: 1uF, Capacitor_SMD:C_0402_1005Metric, symbol Device:C
- removed C15: 100nF, Capacitor_SMD:C_0402_1005Metric, symbol Device:C
- removed J6: 532610671, co2_sensor_footprint:CON_532610671, symbol co2_sensor_molex_footprint:532610671
- removed U1: LM2576HVS-3.3, Package_TO_SOT_SMD:TO-263-5_TabPin3, symbol Regulator_Switching:LM2576HVS-3.3
- removed U4: LM2576HVS-5, Package_TO_SOT_SMD:TO-263-5_TabPin3, symbol Regulator_Switching:LM2576HVS-5
- added U2: LM1084-5.0, lm1084IT_regulator:T03B, symbol Regulator_Linear:LM1084-5.0
- added U3: LM1084-3.3, lm1084IT_regulator:T03B, symbol Regulator_Linear:LM1084-3.3
Connections:
- net +12V: now also U2.3 (VI), U3.3 (VI)
- net +3.3V: now also U3.2 (VO)
- net +5V: now also U2.2 (VO)
- net GND: now also U2.1 (GND), U3.1 (GND)
- no-connect marks 39 -> 38
